Commit message: some changes

File: cvg_sim_gazebo/urdf/quadrotor_sensors.urdf.xacro (robot description, xacro)
@@ -31,3 +31,8 @@
       <origin xyz="0.15 0.0 0.0" rpy="0 ${M_PI/2} 0"/>
     </xacro:generic_camera>
+		<!-- Optional GPU Laser -->
+    <xacro:include filename="$(find drone_simulator)/urdf/laser.xacro" />
+    <xacro:laser name="laser" sim_name="ardrone" parent="base_link" update_rate="60" >
+      <origin xyz="0.15 0.0 0.0" rpy="0 ${M_PI/2} 0"/>
+    </xacro:laser>
 </robot>
